File: kicad/mdb-slave-esp32s3-sim7080g/mdb-slave-esp32s3-sim7080g.kicad_sch (KiCad schematic)
At the start: 81 parts, among them J1 USB_C_Receptacle_USB2.0_16P, J2 JAE_SIM_Card_SF72S006, J3 Conn_01x03_Pin, J4 Conn_Coaxial, J5 Conn_Coaxial, J6 MDB_Connector, J7 Conn_01x03_Pin, J8 Conn_01x04_Pin, Q1 MMBT3904, Q2 MMBT3904, Q3 MMBT3904, Q4 MMBT3904, Q5 MMBT3904, Q6 MMBT3904, Q7 MMBT3904, SW1 SW_Push, U1 ESP32-S3FH4R2, U2 SIM7080G, U3 LM2594HVM-3.3, U4 TLP785, U5 TLP785, Y1 Crystal_GND24

Commit message: chore(kicad): update sim7080g schematic and add hardware project archive
Parts:
- removed AE1: Antenna, RF_Antenna:Texas_SWRA117D_2.4GHz_Left, symbol Device:Antenna
- added C18: 100uF, Capacitor_SMD:CP_Elec_6.3x5.8, symbol Device:C_Polarized
- added C22: 220uF, Capacitor_Tantalum_SMD:CP_EIA-3528-21_Kemet-B, symbol Device:C_Polarized
- added C23, C24, C25, C26, C27, C28: 0.1uF, Capacitor_SMD:C_0603_1608Metric, symbol Device:C
- added D5: D_Schottky, Diode_SMD:D_SOD-123, symbol Device:D_Schottky
- added J10: Conn_Coaxial, Connector_Coaxial:U.FL_Hirose_U.FL-R-SMT-1_Vertical, symbol Connector:Conn_Coaxial
- added J9: SD_Card_Device, symbol Connector:SD_Card_Device
- added L5: 100uH, Inductor_SMD:L_7.3x7.3_H3.5, symbol Device:L
- added Q8, Q9: MMBT3904, Package_TO_SOT_SMD:SOT-23, symbol Transistor_BJT:MMBT3904
- added R26, R29, R31, R32, R33, R34, R35: 10k, Resistor_SMD:R_0603_1608Metric, symbol Device:R
- added R28, R30: 4K7, Resistor_SMD:R_0603_1608Metric, symbol Device:R
- added U6: MAX3232, symbol Interface_UART:MAX3232
- added U7: LM2594HVM-12, Package_SO:SOIC-8_3.9x4.9mm_P1.27mm, symbol Regulator_Switching:LM2594HVM-12
Connections:
- net +3V3: now also C26.1, C27.2, C28.2, J9.4 (VDD), R26.2, R28.1, R29.2, R30.1, R31.1, R32.1, R33.1, R34.1, R35.1, U6.16 (VCC)
- net GND: now also C18.2, C22.2, C25.1, C27.1, C28.1, D5.2 (A), J10.2 (Ext), J9.3 (VSS), J9.6 (VSS), U6.15 (GND), U7.5 (~{ON}/OFF), U7.6 (GND)
- net io1: now also Q8.3 (C), R26.1
- net io2: now also Q9.3 (C), R29.1
- net io7: now also J9.5 (CLK)
- net u0rxd: now also U6.12 (R1OUT)
- net u0txd: now also U6.11 (T1IN)
- net vin: now also C18.1, U7.7 (VIN)
- net at C1.1, L1.2: now also J10.1 (In)
- net io33: now reaches U1.38 (GPIO33)
- net io33: now also J9.7 (DAT0), R31.2
- net io34: now reaches U1.39 (GPIO34)
- net io34: now also J9.8 (DAT1), R33.2
- net io35: now reaches U1.40 (GPIO35)
- net io35: now also J9.9 (DAT2), R34.2
- net io36: now reaches U1.41 (GPIO36)
- net io36: now also J9.1 (CD/DAT3), R35.2
- net io37: now reaches U1.42 (GPIO37)
- net io37: now also J9.2 (CMD), R32.2
- new net: C25.2, U6.6 (VS-)
- new net: D5.1 (K), L5.1, U7.8 (OUT)
- new net: C26.2, U6.2 (VS+)
- new net: Q8.1 (B), R28.2
- new net: C23.1, U6.3 (C1-)
- new net: C23.2, U6.1 (C1+)
- new net: C24.1, U6.5 (C2-)
- new net: C24.2, U6.4 (C2+)
- new net: Q9.1 (B), R30.2
- new net +12V: C22.1, L5.2, U7.4 (FB)
- new net rs232_rx: U6.14 (T1OUT)
- new net rs232_tx: U6.13 (R1IN)
- new net wiegand_data0: Q8.2 (E)
- new net wiegand_data1: Q9.2 (E)
- no-connect marks 31 -> 29
Other:
- moved on the sheet: BZ1, C1, C10, C11, C12, C13, C14, C15, C16, C17, C19, C2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
